File: Control Board/Control Board.kicad_pcb (KiCad board)
At the start: 2 copper layers, 85 x 56 mm, 54 parts, among them J1 Raspberry_Pi_2_3, J9 Conn_01x04_Pin

Commit message: More changes to PCB / Schematic
Schematic complete, PCB in progress
Parts:
- added BAT_IN1: BCH-381H-2GN, Control Board Custom:BCH-381H-2GN, F.Cu at (107.1, 69.0)
- added D1: MBR0580S1, StandardPackages_Custom:SOD-123, F.Cu at (102.9, 96.7)
- added D2: MBR0580S1, StandardPackages_Custom:SOD-123, F.Cu at (102.9, 82.9)
- added D3: SMAJ6.0A, StandardPackages_Custom:DO-214AC, F.Cu at (98.1, 88.3)
- added D4: SMAJ6.0A, StandardPackages_Custom:DO-214AC, F.Cu at (99.3, 102.0)
- added D5: B240AE-13, StandardPackages_Custom:DO-214AC, F.Cu at (66.3, 32.9)
- added D6: LED_Small_Filled, LED_SMD:LED_0805_2012Metric_Pad1.15x1.40mm_HandSolder, F.Cu at (72.2, 40.8)
- added D7: LED_Small_Filled, LED_SMD:LED_0805_2012Metric_Pad1.15x1.40mm_HandSolder, F.Cu at (94.5, 40.8)
- added D8: LED_Small_Filled, LED_SMD:LED_0805_2012Metric_Pad1.15x1.40mm_HandSolder, F.Cu at (92.0, 40.8)
- added EXT_LED1: BCH-381H-2GN, Control Board Custom:BCH-381H-2GN, F.Cu at (107.1, 83.0)
- added PUMP_IN1: BCH-381H-2GN, Control Board Custom:BCH-381H-2GN, F.Cu at (107.1, 97.0)
- added Q1: BSS214NH, StandardPackages_Custom:SOT23-3, F.Cu at (99.6, 98.2)
- added Q2: BSS214NH, StandardPackages_Custom:SOT23-3, F.Cu at (98.8, 84.5)
- added STEMMA1: JST SH, Connector_Adafruit_Custom:Adafruit STEMMA, 4-pin JST SH, F.Cu at (35.9, 92.3)
- added STEMMA2: JST SH, Connector_Adafruit_Custom:Adafruit STEMMA, 4-pin JST SH, F.Cu at (35.8, 73.7)
- added STEMMA4: JST PH, Connector_Adafruit_Custom:Adafruit STEMMA, 3-pin JST PH, F.Cu at (24.2, 21.7)
- added STEMMA5: JST PH, Connector_Adafruit_Custom:Adafruit STEMMA, 3-pin JST PH, F.Cu at (24.1, 38.0)
- added U1: PIC18F16Q41, StandardPackages_Custom:SSOP-20, 5.3mm Body, F.Cu at (61.0, 81.4)
- added U2: PI4ULS5V202UEX, StandardPackages_Custom:MSOP-8, F.Cu at (50.1, 69.5)
- R10, R11: moved to B.Cu
- moved R7 135.9 mm to (72.2, 36.7), turned to -90 degrees
- moved R9 127.7 mm to (92.0, 36.7), turned to 90 degrees
- moved R8 126.2 mm to (94.5, 36.7), turned to 90 degrees
- moved R21 101.6 mm to (96.5, 81.2)
- moved ADDR0 98.0 mm to (65.6, 71.5)
- moved R11 94.0 mm to (39.9, 63.6)
- moved R24 94.0 mm to (99.1, 77.1), turned to 180 degrees
- moved ADDR1 93.3 mm to (65.6, 73.5)
- moved R23 93.2 mm to (102.9, 77.9), turned to -90 degrees
- moved R4 92.6 mm to (57.7, 68.7), turned to 180 degrees
- moved R12 89.3 mm to (97.0, 94.9)
- moved R10 89.1 mm to (39.9, 65.7)
- moved R13 88.4 mm to (96.0, 98.2), turned to -90 degrees
- moved C5 88.0 mm to (52.3, 66.4)
- moved R3 87.8 mm to (57.7, 70.7), turned to 180 degrees
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- renumbered R6 to ADDR0, R5 to ADDR1, ANALOG1_EXT1 to ANALOG_EXT1, ANALOG2_EXT1 to ANALOG_EXT2, J9 to EXT_I2C1
Connections:
- REF** pad 1: (no net) -> GND (x4)
Other:
- board text added: "3.3V"
- board text added: "3.3V Only"
- board text added: "5V"
- board text added: "GND"
- board text added: "PWM"
- board text added: "SCL"
- board text added: "SDA"
- board text added: "VBAT"

Commit message: More work on PCB
Parts:
- removed STEMMA2: JST SH, Connector_Adafruit_Custom:Adafruit STEMMA, 4-pin JST SH
- removed STEMMA5: JST PH, Connector_Adafruit_Custom:Adafruit STEMMA, 3-pin JST PH
- added C15: 220uF, Capacitor_THT:C_Radial_D8.0mm_H11.5mm_P3.50mm, F.Cu at (87.7, 71.2)
- added PTC2: 1.1A, Control Board Custom:0ZCG Series PTC, F.Cu at (100.4, 67.2)
- added PTC3: 100mA, Control Board Custom:0ZCG Series PTC, F.Cu at (57.9, 80.8)
- added RST_SW1: TL6400AF160QJ, Control Board Custom:TL6400AF160QJ, F.Cu at (83.8, 79.5)
- R10, R11: moved to F.Cu
- moved STEMMA4 95.0 mm to (69.6, 105.1), turned to 0 degrees
- moved ANALOG_EXT1 65.0 mm to (72.1, 97.3), turned to -90 degrees
- moved ANALOG_EXT2 52.3 mm to (85.6, 101.3), turned to -90 degrees
- moved D5 45.9 mm to (94.0, 69.5), turned to 90 degrees
- moved R7 44.0 mm to (98.1, 72.3), turned to 0 degrees
- moved D6 43.5 mm to (102.1, 72.3), turned to 180 degrees
- moved SERVO6 39.7 mm to (38.6, 100.8), turned to -90 degrees
- moved C8 39.1 mm to (37.6, 64.7), turned to 0 degrees
- moved C13 38.3 mm to (37.6, 98.0), turned to 0 degrees
- moved R9 37.4 mm to (80.8, 72.4), turned to 0 degrees
- moved R8 36.1 mm to (80.8, 70.1), turned to 0 degrees
- moved R19 35.7 mm to (42.7, 100.8), turned to 0 degrees
- moved SERVO1 35.5 mm to (38.6, 67.6), turned to -90 degrees
- moved D8 35.1 mm to (76.7, 72.4), turned to 0 degrees
- moved D7 34.3 mm to (76.7, 70.1), turned to 0 degrees
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Connections:
- net PI_SCL renamed /PI_SCL
- net PI_SDA renamed /PI_SDA
- J1 pad 1: Net-(J1-3V3-Pad1) -> +3.3V
- J1 pad 17: Net-(J1-3V3-Pad1) -> +3.3V
Routing:
- net VBAT: track 0.00 -> 159.1 mm
- net +5V: track 0.00 -> 71.9 mm
- net SCL: track 0.00 -> 59.1 mm
- net SDA: track 0.00 -> 55.7 mm
- net ICSPCLK: track 0.00 -> 52.5 mm
- net ICSPDAT: track 0.00 -> 49.6 mm
- net ~{MCLR}: track 0.00 -> 44.3 mm
- net +3.3V: track 0.00 -> 43.4 mm
- net GND: track 0.00 -> 39.2 mm, vias 0 -> 5
- net SERVO1: track 0.00 -> 38.7 mm
- net Net-(J1-5V-Pad2): track 0.00 -> 37.1 mm
- net SERVO2: track 0.00 -> 33.3 mm
- net SERVO6: track 0.00 -> 31.7 mm
- net SERVO3: track 0.00 -> 29.8 mm
- net SERVO5: track 0.00 -> 29.1 mm
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- added copper zone on F.Cu, net +5V
- added copper zone on B.Cu, net GND
Other:
- board text added: "AN1"
- board text added: "AN2"
- board text added: "BAT"
- board text added: "DBG0"
- board text added: "DBG1"
- board text added: "Rev ${REVISION}"
- board text removed: "3.3V"
- board text removed: "3.3V Only"

Commit message: Draft of PCB
Parts:
- added EXT_I2C2: Conn_01x04_Pin, Connector_PinHeader_2.54mm:PinHeader_1x04_P2.54mm_Vertical, F.Cu at (48.5, 69.1)
- added G***: LOGO, LOGO, F.Cu at (50.5, 89.4)
- moved D1 15.9 mm to (101.9, 80.8)
- moved D4 15.9 mm to (98.3, 86.1)
- moved Q1 15.9 mm to (98.5, 82.3)
- moved R12 15.9 mm to (96.0, 79.0)
- moved R13 15.9 mm to (95.0, 82.3)
- moved R24 15.6 mm to (99.8, 92.7)
- moved EXT_LED1 14.0 mm to (107.1, 97.0)
- moved PUMP_IN1 14.0 mm to (107.1, 83.0)
- moved D2 13.8 mm to (102.9, 96.8)
- moved D3 13.8 mm to (98.0, 102.1)
- moved Q2 13.8 mm to (98.8, 98.3)
- moved R22 13.8 mm to (95.5, 98.3)
- moved R23 13.8 mm to (102.9, 91.7)
- moved R21 13.8 mm to (96.5, 95.0)
Connections:
- net /PI_SCL renamed PI_SCL
- net /PI_SDA renamed PI_SDA
- U1 pad 11: PUMP_EN -> EXT_LED
- U1 pad 15: EXT_LED -> PUMP_EN
Routing:
- net +5V: track 71.9 -> 134.4 mm, vias 0 -> 3
- net VBAT: track 159.1 -> 173.5 mm
- net GND: track 39.2 -> 51.9 mm, vias 5 -> 7
- net +3.3V: track 43.4 -> 53.1 mm
- net Net-(J1-5V-Pad2): track 37.1 -> 44.5 mm
- net PI_SCL: track 22.9 -> 27.3 mm
- net PI_SDA: track 26.8 -> 29.3 mm
- net Net-(U1-~{MCLR}/VPP/RA3): track 24.3 -> 22.3 mm
- net Net-(D2-PadK): track 10.9 -> 8.93 mm
- net SERVO2: track 33.3 -> 34.3 mm
- net SERVO1: track 38.7 -> 39.7 mm
- net PUMP_EN: track 20.5 -> 21.3 mm, vias 0 -> 2
- net Net-(Q1-D): track 13.5 -> 14.2 mm
- net EXT_LED: track 20.7 -> 20.2 mm, vias 0 -> 2
- added copper zone on F.Cu, net GND
Other:
- board text added: "+"
- board text added: "3.3V"
- board text added: "Designed by Robert Perkel"
- board text added: "Documentation Firmware PCB Files"
- board text added: "Evilia Boat Sampling HAT"
- board text added: "PI_SCL"
- board text added: "PI_SDA"
- board text added: "The Pink Flamingo"

Commit message: Finished PCB
Parts:
- added G***: LOGO, LOGO, B.Cu at (72.9, 69.3)
Routing:
- net +5V: track 134.4 -> 136.3 mm
Other:
- board text added: "Pullup MCU"
- board text added: "Pullup Rasp. Pi"
- board text added: "SERVO1"
- board text added: "SERVO2"
- board text added: "SERVO3"
- board text added: "SERVO4"
- board text added: "SERVO5"
- board text added: "SERVO6"
- board text added: "The Salty Flamingo 1"
- board text removed: "The Pink Flamingo"

Commit message: Added DAC2 for Self-Testing. Updated PCB/SCH to Rev A2
Increased size of pads for reset switch. Added debug header for OPAMP. Added pin 1 marker for programming.
Parts:
- added OPAMP_TEST1: Conn_01x02_Pin, Connector_PinHeader_2.54mm:PinHeader_1x02_P2.54mm_Vertical, F.Cu at (76.5, 92.7)
- BAT_IN1, EXT_LED1, PUMP_IN1: value BCH-381H-2GN -> BCH-381H-2 GN
Connections:
- U1 pad 14: unconnected-(U1-RC2-Pad14) -> OPAMP_OUT
Routing:
- net OPAMP_OUT: track 0.00 -> 6.88 mm
- net Net-(U1-RB5): track 16.1 -> 14.9 mm, vias 0 -> 1
- net GND: vias 7 -> 6
Other:
- board text added: "OPAMP"

Commit message: PCB fixes
Routing:
- net Net-(J1-5V-Pad2): track 44.5 -> 39.6 mm
- net PI_SCL: track 27.3 -> 25.9 mm
- net Net-(Q1-D): track 14.2 -> 13.1 mm
- net GND: vias 6 -> 7
- net Net-(U1-RB5): vias 1 -> 0
Changed lines of the file:
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@@
   )
   (segment (start 36.576 61.722) (end 36.576 59.034) (width 0.1524) (layer "F.Cu") (net 1))
-  (segment (start 55.297 75.617) (end 55.297 80.518) (width 0.1524) (layer "F.Cu") (net 1))
   (segment (start 38.608 63.754) (end 36.576 61.722) (width 0.1524) (layer "F.Cu") (net 1))
   (segment (start 45.72 76.454) (end 45.72 67.564) (width 0.1524) (layer "F.Cu") (net 1))
@@
   (segment (start 95.594 99.348) (end 95.52 99.274) (width 0.508) (layer "F.Cu") (net 2))
   (segment (start 78.9 83.66) (end 77.768 83.66) (width 0.254) (layer "F.Cu") (net 2))
-  (segment (start 97.478 83.296) (end 97.528 83.246) (width 0.508) (layer "F.Cu") (net 2))
   (segment (start 56.388 70.866) (end 56.388 71.628) (width 0.254) (layer "F.Cu") (net 2))
   (segment (start 103.161 72.272) (end 105.751 72.272) (width 0.508) (layer "F.Cu") (net 2))
@@
   (segment (start 86.52 79.502) (end 88.646 79.502) (width 0.508) (layer "F.Cu") (net 2))
   (segment (start 92.964 101.346) (end 93.702 102.084) (width 0.508) (layer "F.Cu") (net 2))
+  (via (at 74.168 93.98) (size 0.8) (drill 0.4) (layers "F.Cu" "B.Cu") (net 2))
   (via (at 92.964 101.346) (size 0.8) (drill 0.4) (layers "F.Cu" "B.Cu") (net 2))
   (via (at 84.328 88.392) (size 0.8) (drill 0.4) (layers "F.Cu" "B.Cu") (net 2))
@@
   (segment (start 38.6145 64.718) (end 38.608 64.7245) (width 0.1524) (layer "B.Cu") (net 29))
   (segment (start 36.038 94.182) (end 36.038 100.786) (width 0.508) (layer "F.Cu") (net 30))
-  (segment (start 106.773 81.44) (end 107.118 81.095) (width 0.508) (layer "F.Cu") (net 30))
   (segment (start 109.474 86.614) (end 109.474 83.312) (width 0.508) (layer "F.Cu") (net 30))
   (segment (start 36.068 67.564) (end 36.068 74.114) (width 0.508) (layer "F.Cu") (net 30))
@@
   (segment (start 77.232 79.502) (end 76.962 79.232) (width 0.1524) (layer "F.Cu") (net 41))
   (segment (start 76.946 81.28) (end 76.946 81.042) (width 0.1524) (layer "F.Cu") (net 41))
-  (segment (start 81.12 79.248) (end 80.866 79.502) (width 0.1524) (layer "F.Cu") (net 41))
   (segment (start 76.708 67.056) (end 76.708 73.914) (width 0.1524) (layer "F.Cu") (net 41))
   (segment (start 84.3852 63.4428) (end 103.0912 63.4428) (width 0.1524) (layer "F.Cu") (net 42))
@@
   (segment (start 70.568 88.889) (end 50.557 88.889) (width 0.1524) (layer "F.Cu") (net 58))
   (segment (start 70.568 89.539) (end 54.904 89.539) (width 0.1524) (layer "F.Cu") (net 59))
-  (segment (start 43.555 100.684) (end 43.657 100.786) (width 0.1524) (layer "F.Cu") (net 59))
   (segment (start 54.904 89.539) (end 43.657 100.786) (width 0.1524) (layer "F.Cu") (net 59))
+  (segment (start 70.6065 93.98) (end 70.6065 93.7315) (width 0.1524) (layer "F.Cu") (net 60))
   (segment (start 76.921 85.639) (end 77.768 85.639) (width 0.1524) (layer "F.Cu") (net 60))
-  (segment (start 70.6065 93.98) (end 70.6065 93.2235) (width 0.1524) (layer "F.Cu") (net 60))
-  (segment (start 76.2 86.36) (end 76.921 85.639) (width 0.1524) (layer "F.Cu") (net 60))
-  (segment (start 70.6065 93.2235) (end 76.2 87.63) (width 0.1524) (layer "F.Cu") (net 60))
-  (segment (start 76.2 87.63) (end 76.2 86.36) (width 0.1524) (layer "F.Cu") (net 60))
+  (segment (start 75.184 87.376) (end 76.921 85.639) (width 0.1524) (layer "F.Cu") (net 60))
+  (segment (start 70.6065 93.7315) (end 75.184 89.154) (width 0.1524) (layer "F.Cu") (net 60))
+  (segment (start 75.184 89.154) (end 75.184 87.376) (width 0.1524) (layer "F.Cu") (net 60))
   (segment (start 68.58 93.98) (end 70.6065 93.98) (width 0.1524) (layer "F.Cu") (net 60))
   (segment (start 78.617 89.539) (end 83.312 94.234) (width 0.1524) (layer "F.Cu") (net 61))
   (segment (start 94.718 94.972) (end 95.52 94.972) (width 0.1524) (layer "F.Cu") (net 61))
-  (segment (start 95.384 94.836) (end 95.52 94.972) (width 0.1524) (layer "F.Cu") (net 61))
   (segment (start 83.312 94.234) (end 90.678 94.234) (width 0.1524) (layer "F.Cu") (net 61))
   (segment (start 93.98 94.234) (end 94.718 94.972) (width 0.1524) (layer "F.Cu") (net 61))
@@
   (segment (start 76.454 90.17) (end 77.5802 91.2962) (width 0.1524) (layer "F.Cu") (net 63))
   (segment (start 76.7656 88.889) (end 76.454 89.2006) (width 0.1524) (layer "F.Cu") (net 63))
-  (via (at 78.232 94.996) (size 0.8) (drill 0.4) (layers "F.Cu" "B.Cu") (net 63))
   (segment (start 77.768 87.589) (end 76.7656 87.589) (width 0.1524) (layer "F.Cu") (net 64))
   (segment (start 76.7656 87.589) (end 75.692 88.6626) (width 0.1524) (layer "F.Cu") (net 64))
@@
   (segment (start 75.692 91.948) (end 76.454 92.71) (width 0.1524) (layer "F.Cu") (net 64))
   (segment (start 99.528 82.296) (end 101.83 82.296) (width 0.508) (layer "F.Cu") (net 65))
-  (segment (start 101.854 82.272) (end 101.6 82.526) (width 0.508) (layer "F.Cu") (net 65))
   (segment (start 105.917 86.106) (end 100.748 86.106) (width 0.508) (layer "F.Cu") (net 65))
   (segment (start 107.118 84.905) (end 105.917 86.106) (width 0.508) (layer "F.Cu") (net 65))
   (segment (start 101.83 82.296) (end 101.854 82.272) (width 0.508) (layer "F.Cu") (net 65))
   (segment (start 101.6 85.254) (end 100.748 86.106) (width 0.508) (layer "F.Cu") (net 65))
-  (segment (start 106.653 84.44) (end 107.118 84.905) (width 0.508) (layer "F.Cu") (net 65))
   (segment (start 101.6 82.526) (end 101.6 85.254) (width 0.508) (layer "F.Cu") (net 65))
   (segment (start 102.87 98.25) (end 99.83 98.25) (width 0.508) (layer "F.Cu") (net 66))
@@
   (segment (start 102.87 95.25) (end 106.963 95.25) (width 0.508) (layer "F.Cu") (net 69))
   (segment (start 57.038 66.422) (end 57.038 71.628) (width 0.1524) (layer "F.Cu") (net 70))
-  (segment (start 43.455 59.775) (end 43.455 60.473) (width 0.1524) (layer "F.Cu") (net 70))
-  (segment (start 57.038 71.628) (end 57.038 71.008) (width 0.1524) (layer "F.Cu") (net 70))
-  (segment (start 43.455 59.775) (end 43.519 59.775) (width 0.1524) (layer "F.Cu") (net 70))
   (segment (start 43.455 60.473) (end 48.514 65.532) (width 0.1524) (layer "F.Cu") (net 70))
   (segment (start 48.514 65.532) (end 48.514 69.088) (width 0.1524) (layer "F.Cu") (net 70))
